File: CapteursNumerique/CapteursNumerique.kicad_pcb (KiCad board)
At the start: 2 copper layers, 40 x 39 mm, 57 parts, among them J1 EXT-CON, J10 Conn IO, J11 DIS LED, J12 Conn IO, J13 DIS LED, J14 Conn IO, J15 DIS LED, J16 Conn IO, J17 DIS LED, J18 A2, J19 A1, J2 Conn IO, J20 A0, J3 DIS LED, J4 Conn IO, J5 DIS LED, J6 Conn IO, J7 DIS LED, J8 Conn IO, J9 DIS LED, U1 PCF8574

Commit message: Capteurs num production
Parts:
- C2: value 1u -> 10u
- J11, J13, J15, J17, J3, J5, J7, J9: footprint Jumper:SolderJumper-2_P1.3mm_Bridged2Bar_Pad1.0x1.5mm -> Jumper:SolderJumper-2_P1.3mm_Open_Pad1.0x1.5mm
Other:
- board text added: "TOR 2020"
- board text removed: "IOs TOR 2020"
