File: CapteursNumerique/CapteursNumerique.sch (KiCad schematic (older format))
At the start: 15 parts, among them J1 EXT-CON, J18 A2, J19 A1, J20 A0, U1 PCF8574

Commit message: Capteurs num production
Parts:
- C1: LCSC Part (none) -> C28233
- C2: value 1u -> 10u; LCSC Part (none) -> C134721
- D1: LCSC Part (none) -> C72037
- D10: LCSC Part (none) -> C63855
- J1, J18, J19, J20: JLCPCB BOM (none) -> 0
- R1, R22: LCSC Part (none) -> C17471
- R2: LCSC Part (none) -> C17414
- U1: LCSC Part (none) -> C7605
Other:
- moved on the sheet: J1
Changed lines of the file:
@@
 F 2 "Package_SO:SOIC-16W_7.5x10.3mm_P1.27mm" H 3850 3940 50  0001 C CNN
 F 3 "http://www.nxp.com/documents/data_sheet/PCF8574_PCF8574A.pdf" H 3850 3940 50  0001 C CNN
+F 4 "C7605" H 3850 3940 50  0001 C CNN "LCSC Part"
 	1    3850 3940
 	1    0    0    -1
@@
 F 2 "Resistor_SMD:R_0805_2012Metric_Pad1.20x1.40mm_HandSolder" V 1910 3590 50  0001 C CNN
 F 3 "~" H 1870 3600 50  0001 C CNN
+F 4 "C17414" H 1870 3600 50  0001 C CNN "LCSC Part"
 	1    1870 3600
 	1    0    0    -1
@@
 F 2 "LED_SMD:LED_0805_2012Metric_Pad1.15x1.40mm_HandSolder" H 1600 4110 50  0001 C CNN
 F 3 "~" H 1600 4110 50  0001 C CNN
+F 4 "C72037" V 1600 4110 50  0001 C CNN "LCSC Part"
 	1    1600 4110
 	0    -1   -1   0
@@
 F 2 "Resistor_SMD:R_0805_2012Metric_Pad1.20x1.40mm_HandSolder" V 1640 3600 50  0001 C CNN
 F 3 "~" H 1600 3610 50  0001 C CNN
+F 4 "C17471" H 1600 3610 50  0001 C CNN "LCSC Part"
 	1    1600 3610
 	1    0    0    -1
@@
 F 2 "Capacitor_SMD:C_0805_2012Metric_Pad1.18x1.45mm_HandSolder" H 2838 1720 50  0001 C CNN
 F 3 "~" H 2800 1870 50  0001 C CNN
+F 4 "C28233" H 2800 1870 50  0001 C CNN "LCSC Part"
 	1    2800 1870
 	1    0    0    -1
@@
 P 3270 1870
 F 0 "C2" H 3385 1916 50  0000 L CNN
-F 1 "1u" H 3385 1825 50  0000 L CNN
+F 1 "10u" H 3385 1825 50  0000 L CNN
 F 2 "Capacitor_SMD:CP_Elec_4x5.4" H 3270 1870 50  0001 C CNN
 F 3 "~" H 3270 1870 50  0001 C CNN
+F 4 "C134721" H 3270 1870 50  0001 C CNN "LCSC Part"
 	1    3270 1870
 	1    0    0    -1
@@
 Découplage
 Wire Wire Line
-	2750 6040 2580 6040
-Wire Wire Line
-	3250 6040 3430 6040
-Wire Wire Line
-	3430 6440 3250 6440
-Wire Wire Line
-	2750 6440 2580 6440
-Wire Wire Line
-	2750 6240 2580 6240
-NoConn ~ 2750 6140
-NoConn ~ 2750 6340
-NoConn ~ 3250 6340
-NoConn ~ 3250 6240
-NoConn ~ 3250 6140
+	2750 6060 2580 6060
+Wire Wire Line
+	3250 6060 3430 6060
+Wire Wire Line
+	3430 6460 3250 6460
+Wire Wire Line
+	2750 6460 2580 6460
+Wire Wire Line
+	2750 6260 2580 6260
+NoConn ~ 2750 6160
+NoConn ~ 2750 6360
+NoConn ~ 3250 6360
+NoConn ~ 3250 6260
+NoConn ~ 3250 6160
 Text Label 2970 3540 0    50   ~ 0
 SCL
 Text Label 2970 3640 0    50   ~ 0
 SDA
-Text Label 3430 6440 2    50   ~ 0
+Text Label 3430 6460 2    50   ~ 0
 SCL
-Text Label 2580 6440 0    50   ~ 0
+Text Label 2580 6460 0    50   ~ 0
 SDA
 $Comp
 L power:GND #PWR0109
 U 1 1 5FC470EC
-P 3430 5990
-F 0 "#PWR0109" H 3430 5740 50  0001 C CNN
-F 1 "GND" H 3435 5817 50  0000 C CNN
-F 2 "" H 3430 5990 50  0001 C CNN
-F 3 "" H 3430 5990 50  0001 C CNN
-	1    3430 5990
+P 3430 6010
+F 0 "#PWR0109" H 3430 5760 50  0001 C CNN
+F 1 "GND" H 3435 5837 50  0000 C CNN
+F 2 "" H 3430 6010 50  0001 C CNN
+F 3 "" H 3430 6010 50  0001 C CNN
+	1    3430 6010
 	-1   0    0    1
 $EndComp
 Wire Wire Line
-	3430 6040 3430 5990
+	3430 6060 3430 6010
 $Comp
 L power:+5V #PWR0110
 U 1 1 5FC4923D
-P 2580 5990
-F 0 "#PWR0110" H 2580 5840 50  0001 C CNN
-F 1 "+5V" H 2595 6163 50  0000 C CNN
-F 2 "" H 2580 5990 50  0001 C CNN
-F 3 "" H 2580 5990 50  0001 C CNN
-	1    2580 5990
-	1    0    0    -1
-$EndComp
-Wire Wire Line
-	2580 6040 2580 5990
+P 2580 6010
+F 0 "#PWR0110" H 2580 5860 50  0001 C CNN
+F 1 "+5V" H 2595 6183 50  0000 C CNN
+F 2 "" H 2580 6010 50  0001 C CNN
+F 3 "" H 2580 6010 50  0001 C CNN
+	1    2580 6010
+	1    0    0    -1
+$EndComp
+Wire Wire Line
+	2580 6060 2580 6010
 $Comp
 L power:PWR_FLAG #FLG0101
@@
 Wire Wire Line
 	2970 3540 3350 3540
-Text Label 2580 6240 0    50   ~ 0
+Text Label 2580 6260 0    50   ~ 0
 IRQ
-Text Notes 2740 5630 0    50   ~ 0
+Text Notes 2740 5650 0    50   ~ 0
 Interface de \nconnection HE10
 Wire Notes Line
-	2450 5400 2450 6610
-Wire Notes Line
-	2450 6610 3610 6610
-Wire Notes Line
-	3610 6610 3610 5400
-Wire Notes Line
-	3610 5400 2450 5400
+	2450 5420 2450 6630
+Wire Notes Line
+	2450 6630 3610 6630
+Wire Notes Line
+	3610 6630 3610 5420
+Wire Notes Line
+	3610 5420 2450 5420
 Wire Wire Line
 	1870 4340 3350 4340
@@
 F 2 "Jumper:SolderJumper-2_P1.3mm_Open_Pad1.0x1.5mm" H 2450 4660 50  0001 C CNN
 F 3 "~" H 2450 4660 50  0001 C CNN
+F 4 "0" V 2450 4660 50  0001 C CNN "JLCPCB BOM"
 	1    2450 4660
 	0    1    1    0
@@
 F 2 "Jumper:SolderJumper-2_P1.3mm_Open_Pad1.0x1.5mm" H 2740 4660 50  0001 C CNN
 F 3 "~" H 2740 4660 50  0001 C CNN
+F 4 "0" V 2740 4660 50  0001 C CNN "JLCPCB BOM"
 	1    2740 4660
 	0    1    1    0
@@
 F 2 "Jumper:SolderJumper-2_P1.3mm_Open_Pad1.0x1.5mm" H 2170 4660 50  0001 C CNN
 F 3 "~" H 2170 4660 50  0001 C CNN
+F 4 "0" V 2170 4660 50  0001 C CNN "JLCPCB BOM"
 	1    2170 4660
 	0    1    1    0
@@
 L Connector_Generic:Conn_02x05_Odd_Even J1
 U 1 1 5FB3B612
-P 2950 6240
-F 0 "J1" H 3000 6657 50  0000 C CNN
-F 1 "EXT-CON" H 3000 6566 50  0000 C CNN
-F 2 "Connector_IDC:IDC-Header_2x05_P2.54mm_Vertical" H 2950 6240 50  0001 C CNN
-F 3 "~" H 2950 6240 50  0001 C CNN
-	1    2950 6240
+P 2950 6260
+F 0 "J1" H 3000 6677 50  0000 C CNN
+F 1 "EXT-CON" H 3000 6586 50  0000 C CNN
+F 2 "Connector_IDC:IDC-Header_2x05_P2.54mm_Vertical" H 2950 6260 50  0001 C CNN
+F 3 "~" H 2950 6260 50  0001 C CNN
+F 4 "0" H 2950 6260 50  0001 C CNN "JLCPCB BOM"
+	1    2950 6260
 	1    0    0    -1
 $EndComp
@@
 F 2 "Resistor_SMD:R_0805_2012Metric_Pad1.20x1.40mm_HandSolder" V 2160 1630 50  0001 C CNN
 F 3 "~" H 2120 1640 50  0001 C CNN
+F 4 "C17471" H 2120 1640 50  0001 C CNN "LCSC Part"
 	1    2120 1640
 	1    0    0    -1
@@
 F 2 "LED_SMD:LED_0805_2012Metric_Pad1.15x1.40mm_HandSolder" H 2120 1960 50  0001 C CNN
 F 3 "~" H 2120 1960 50  0001 C CNN
+F 4 "C63855" V 2120 1960 50  0001 C CNN "LCSC Part"
 	1    2120 1960
 	0    -1   -1   0

Commit message: Module alim ISO, clean master alim
Parts:
- R3, R4, R5: LCSC Part (none) -> C17414
Changed lines of the file:
@@
 F 2 "Resistor_SMD:R_0805_2012Metric_Pad1.20x1.40mm_HandSolder" V 2490 3580 50  0001 C CNN
 F 3 "~" H 2450 3590 50  0001 C CNN
+F 4 "C17414" H 2450 3590 50  0001 C CNN "LCSC Part"
 	1    2450 3590
 	1    0    0    -1
@@
 F 2 "Resistor_SMD:R_0805_2012Metric_Pad1.20x1.40mm_HandSolder" V 2210 3580 50  0001 C CNN
 F 3 "~" H 2170 3590 50  0001 C CNN
+F 4 "C17414" H 2170 3590 50  0001 C CNN "LCSC Part"
 	1    2170 3590
 	1    0    0    -1
@@
 F 2 "Resistor_SMD:R_0805_2012Metric_Pad1.20x1.40mm_HandSolder" V 2780 3590 50  0001 C CNN
 F 3 "~" H 2740 3600 50  0001 C CNN
+F 4 "C17414" H 2740 3600 50  0001 C CNN "LCSC Part"
 	1    2740 3600
 	1    0    0    -1
