File: Alimentation/ModuleMesureDemi/ModuleMesureDemi.sch (KiCad schematic (older format))
At the start: 71 parts, among them J1 Out Mes 2, J10 I2C SDA, J11 SWD, J12 ARIG Interf, J2 In Mes 1, J3 Out Mes 1, J4 In Mes 2, J5 Out Mes 3, J6 Out Mes 4, J7 In Mes 3, J8 In Mes 4, J9 I2C SCL, Q1 BSS138, Q2 BSS138, SW1 Reset, SW2 Boot0, SW3 Boot1, U1 ACS711xEXLT-15AB, U2 ACS711xEXLT-15AB, U3 ACS711xEXLT-15AB, U4 ACS711xEXLT-15AB, U5 AMS1117-3.3, U6 STM32F103C8Tx, Y1 16Mhz

Commit message: Finalisation pour commande pack Alimentation 14/02/2021
Parts:
- removed C3, C4: 100n, Capacitor_SMD:C_0402_1005Metric_Pad0.74x0.62mm_HandSolder, symbol Device:C_Small
- removed J1: Out Mes 2, TerminalBlock_Phoenix:TerminalBlock_Phoenix_MKDS-1,5-3-5.08_1x03_P5.08mm_Horizontal, symbol Connector:Screw_Terminal_01x03
- removed J2: In Mes 1, TerminalBlock_Phoenix:TerminalBlock_Phoenix_MKDS-1,5-2-5.08_1x02_P5.08mm_Horizontal, symbol Connector:Screw_Terminal_01x02
- removed J3: Out Mes 1, TerminalBlock_Phoenix:TerminalBlock_Phoenix_MKDS-1,5-3-5.08_1x03_P5.08mm_Horizontal, symbol Connector:Screw_Terminal_01x03
- removed J4: In Mes 2, TerminalBlock_Phoenix:TerminalBlock_Phoenix_MKDS-1,5-2-5.08_1x02_P5.08mm_Horizontal, symbol Connector:Screw_Terminal_01x02
- removed R11, R14: 10k, Resistor_SMD:R_0805_2012Metric_Pad1.20x1.40mm_HandSolder, symbol Device:R_Small
- removed R5, R7: 5.6k, Resistor_SMD:R_0805_2012Metric_Pad1.20x1.40mm_HandSolder, symbol Device:R_Small
- removed R6, R8: 1.8k, Resistor_SMD:R_0805_2012Metric_Pad1.20x1.40mm_HandSolder, symbol Device:R_Small
- removed U1, U2: ACS711xEXLT-15AB, Sensor_Current:Allegro_QFN-12-10-1EP_3x3mm_P0.5mm, symbol Sensor_Current:ACS711xEXLT-15AB
- added J1: 5V, TerminalBlock_Phoenix:TerminalBlock_Phoenix_MPT-0,5-2-2.54_1x02_P2.54mm_Horizontal, symbol Connector:Screw_Terminal_01x02
- added JP1: ADD1, Jumper:SolderJumper-3_P1.3mm_Open_RoundedPad1.0x1.5mm, symbol Jumper:SolderJumper_3_Open
- added JP2: ADD2, Jumper:SolderJumper-3_P1.3mm_Open_RoundedPad1.0x1.5mm, symbol Jumper:SolderJumper_3_Open
- added JP3: ADD3, Jumper:SolderJumper-3_P1.3mm_Open_RoundedPad1.0x1.5mm, symbol Jumper:SolderJumper_3_Open
- C1, C10, C12, C13, C14, C15, C18, C2, C9: LCSC Part C541405 -> C1525; Tension 6.3V -> 16V
- C11: LCSC Part C87147 -> C23733; Tension 6.3V -> 10V
- C16: LCSC Part C87144 -> C52923; Tension 6.3V -> 25V
- C17: LCSC Part C309453 -> C15195; Tension 6.3V -> 50V
- C5: footprint Capacitor_SMD:CP_Elec_5x5.4 -> Capacitor_SMD:CP_Elec_5x5.3; LCSC Part C72472 -> C249463
- C6: LCSC Part C58276 -> C249900
- C7, C8: LCSC Part (none) -> C1547; Tension 6.3V -> 50V
- D1, D2: value LED_Small -> Green; LCSC Part (none) -> C63855
- H1, H2, H3, H4, J10, J12, J9: JLCPCB BOM (none) -> 0
- J11: footprint Connector_PinHeader_1.27mm:PinHeader_2x05_P1.27mm_Vertical_SMD -> Connector_PinHeader_1.27mm:PinHeader_2x05_P1.27mm_Vertical; JLCPCB BOM (none) -> 0
- J5: value Out Mes 3 -> Out Mes 1; JLCPCB BOM (none) -> 0
- J6: value Out Mes 4 -> Out Mes 2; JLCPCB BOM (none) -> 0
- J7: value In Mes 3 -> In Mes 1; JLCPCB BOM (none) -> 0
- J8: value In Mes 4 -> In Mes 2; JLCPCB BOM (none) -> 0
- L1: LCSC Part (none) -> C26443
- Q1, Q2: LCSC Part (none) -> C112239
- R1, R3: LCSC Part (none) -> C26024
- R10, R12, R13, R15, R16, R18, R19, R22, R9: LCSC Part (none) -> C17414
- R17: value 18 -> 33; LCSC Part (none) -> C17634
- R2, R4: LCSC Part (none) -> C17398
- R20: LCSC Part (none) -> C25118
- R21: value 1k5 -> 33; LCSC Part (none) -> C17634
- U5: LCSC Part (none) -> C6186
Connections:
- net labels added: ADD1, ADD2, ADD3
- net labels removed: +12C, +12L, ANA_CURRENT_3, ANA_CURRENT_4, ANA_VOLT_3, ANA_VOLT_4, FAULT_3, FAULT_4, OutMes3, OutMes4
- wire segments 214 -> 172
- no-connect marks 40 -> 35
Other:
- moved on the sheet: C1, C2, J10, J11, J12, J5, J6, J7, J8, J9, R1, R10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
