File: InterfaceRaspi/ConvertLvHv.sch (KiCad schematic (older format))
At the start: 3 parts, among them Q1 BSS138

Commit message: Finalisation interface Raspi
Parts:
- Q1: LCSC Part C112239 -> C426569
Changed lines of the file:
@@
 F 2 "Package_TO_SOT_SMD:SOT-23" H 6200 3475 50  0001 L CIN
 F 3 "https://www.onsemi.com/pub/Collateral/BSS138-D.PDF" H 6000 3550 50  0001 L CNN
-F 4 "C112239" V 6000 3550 50  0001 C CNN "LCSC Part"
+F 4 "C426569" V 6000 3550 50  0001 C CNN "LCSC Part"
 	1    6000 3550
 	0    1    1    0
