File: InterfaceRaspi/InterfaceRaspi.kicad_pcb (KiCad board)
At the start: 4 copper layers, 65 x 56 mm, 50 parts, among them J1 Interf 5, J10 I2C 5V, J11 I2C 5V, J2 Interf 7, J3 Interf 1, J4 Interf 3, J5 Interf 6, J6 Interf RGB, J7 Interf 2, J8 Interf 4, J9 Raspberry_Pi_2_3, Q1 BSS138, Q10 BSS138, Q11 BSS138, Q2 BSS138, Q3 BSS138, Q4 BSS138, Q5 BSS138, Q6 BSS138, Q7 BSS138, Q8 BSS138, Q9 BSS138

Commit message: Finalisation interf Raspi
Parts:
- added G***: LOGO, ARIG:Logo_ARIG_12_6x6_6, B.Cu at (113.0, 124.2)
