File: InterfaceRaspi/InterfaceRaspi.sch (KiCad schematic (older format))
At the start: 17 parts, among them J1 Interf 5, J10 I2C 5V, J11 I2C 5V, J2 Interf 7, J3 Interf 1, J4 Interf 3, J5 Interf 6, J6 Interf RGB, J7 Interf 2, J8 Interf 4, J9 Raspberry_Pi_2_3

Commit message: Finalisation interf Raspi
Parts:
- H1, H2, H3, H4, J1, J10, J11, J2, J3, J4, J5, J6, J7, J8, J9: LCSC Part (none) -> 0
- R24, R25: LCSC Part (none) -> C17673
Changed lines of the file:
@@
 F 2 "Connector_PinSocket_2.54mm:PinSocket_2x20_P2.54mm_Vertical" H 9230 3770 50  0001 C CNN
 F 3 "https://www.raspberrypi.org/documentation/hardware/raspberrypi/schematics/rpi_SCH_3bplus_1p0_reduced.pdf" H 9230 3770 50  0001 C CNN
+F 4 "0" H 9230 3770 50  0001 C CNN "LCSC Part"
 	1    9230 3770
 	1    0    0    -1
@@
 F 2 "Connector_IDC:IDC-Header_2x05_P2.54mm_Vertical" H 1460 1430 50  0001 C CNN
 F 3 "~" H 1460 1430 50  0001 C CNN
+F 4 "0" H 1460 1430 50  0001 C CNN "LCSC Part"
 	1    1460 1430
 	1    0    0    -1
@@
 F 2 "Connector_IDC:IDC-Header_2x05_P2.54mm_Vertical" H 2730 1430 50  0001 C CNN
 F 3 "~" H 2730 1430 50  0001 C CNN
+F 4 "0" H 2730 1430 50  0001 C CNN "LCSC Part"
 	1    2730 1430
 	1    0    0    -1
@@
 F 2 "Connector_IDC:IDC-Header_2x05_P2.54mm_Vertical" H 1460 2360 50  0001 C CNN
 F 3 "~" H 1460 2360 50  0001 C CNN
+F 4 "0" H 1460 2360 50  0001 C CNN "LCSC Part"
 	1    1460 2360
 	1    0    0    -1
@@
 F 2 "Connector_IDC:IDC-Header_2x05_P2.54mm_Vertical" H 2730 2360 50  0001 C CNN
 F 3 "~" H 2730 2360 50  0001 C CNN
+F 4 "0" H 2730 2360 50  0001 C CNN "LCSC Part"
 	1    2730 2360
 	1    0    0    -1
@@
 F 2 "Connector_IDC:IDC-Header_2x05_P2.54mm_Vertical" H 1430 3250 50  0001 C CNN
 F 3 "~" H 1430 3250 50  0001 C CNN
+F 4 "0" H 1430 3250 50  0001 C CNN "LCSC Part"
 	1    1430 3250
 	1    0    0    -1
@@
 F 2 "Connector_IDC:IDC-Header_2x05_P2.54mm_Vertical" H 2700 3250 50  0001 C CNN
 F 3 "~" H 2700 3250 50  0001 C CNN
+F 4 "0" H 2700 3250 50  0001 C CNN "LCSC Part"
 	1    2700 3250
 	1    0    0    -1
@@
 F 2 "Connector_IDC:IDC-Header_2x05_P2.54mm_Vertical" H 1430 4180 50  0001 C CNN
 F 3 "~" H 1430 4180 50  0001 C CNN
+F 4 "0" H 1430 4180 50  0001 C CNN "LCSC Part"
 	1    1430 4180
 	1    0    0    -1
@@
 F 2 "Connector_IDC:IDC-Header_2x05_P2.54mm_Vertical" H 2700 4180 50  0001 C CNN
 F 3 "~" H 2700 4180 50  0001 C CNN
+F 4 "0" H 2700 4180 50  0001 C CNN "LCSC Part"
 	1    2700 4180
 	1    0    0    -1
@@
 F 2 "MountingHole:MountingHole_3.2mm_M3_ISO14580_Pad" H 2540 5160 50  0001 C CNN
 F 3 "~" H 2540 5160 50  0001 C CNN
+F 4 "0" H 2540 5160 50  0001 C CNN "LCSC Part"
 	1    2540 5160
 	0    1    1    0
@@
 F 2 "MountingHole:MountingHole_3.2mm_M3_ISO14580_Pad" H 2540 5340 50  0001 C CNN
 F 3 "~" H 2540 5340 50  0001 C CNN
+F 4 "0" H 2540 5340 50  0001 C CNN "LCSC Part"
 	1    2540 5340
 	0    1    1    0
@@
 F 2 "MountingHole:MountingHole_3.2mm_M3_ISO14580_Pad" H 2540 5520 50  0001 C CNN
 F 3 "~" H 2540 5520 50  0001 C CNN
+F 4 "0" H 2540 5520 50  0001 C CNN "LCSC Part"
 	1    2540 5520
 	0    1    1    0
@@
 F 2 "MountingHole:MountingHole_3.2mm_M3_ISO14580_Pad" H 2540 5710 50  0001 C CNN
 F 3 "~" H 2540 5710 50  0001 C CNN
+F 4 "0" H 2540 5710 50  0001 C CNN "LCSC Part"
 	1    2540 5710
 	0    1    1    0
@@
 F 2 "TerminalBlock_Phoenix:TerminalBlock_Phoenix_MPT-0,5-2-2.54_1x02_P2.54mm_Horizontal" H 4890 1240 50  0001 C CNN
 F 3 "~" H 4890 1240 50  0001 C CNN
+F 4 "0" H 4890 1240 50  0001 C CNN "LCSC Part"
 	1    4890 1240
 	1    0    0    -1
@@
 F 2 "Resistor_SMD:R_0805_2012Metric_Pad1.20x1.40mm_HandSolder" H 4290 960 50  0001 C CNN
 F 3 "~" H 4290 960 50  0001 C CNN
+F 4 "C17673" H 4290 960 50  0001 C CNN "LCSC Part"
 	1    4290 960
 	1    0    0    -1
@@
 F 2 "Resistor_SMD:R_0805_2012Metric_Pad1.20x1.40mm_HandSolder" H 4570 960 50  0001 C CNN
 F 3 "~" H 4570 960 50  0001 C CNN
+F 4 "C17673" H 4570 960 50  0001 C CNN "LCSC Part"
 	1    4570 960
 	1    0    0    -1
@@
 F 2 "TerminalBlock_Phoenix:TerminalBlock_Phoenix_MPT-0,5-2-2.54_1x02_P2.54mm_Horizontal" H 4690 2750 50  0001 C CNN
 F 3 "~" H 4690 2750 50  0001 C CNN
+F 4 "0" H 4690 2750 50  0001 C CNN "LCSC Part"
 	1    4690 2750
 	1    0    0    -1

Commit message: Finalisation interface Raspi
Parts:
- H1, H2, H3, H4, J1, J10, J11, J2, J3, J4, J5, J6, J7, J8, J9: JLCPCB BOM (none) -> 0; LCSC Part 0 -> (none)
Changed lines of the file:
@@
 F 2 "Connector_PinSocket_2.54mm:PinSocket_2x20_P2.54mm_Vertical" H 9230 3770 50  0001 C CNN
 F 3 "https://www.raspberrypi.org/documentation/hardware/raspberrypi/schematics/rpi_SCH_3bplus_1p0_reduced.pdf" H 9230 3770 50  0001 C CNN
-F 4 "0" H 9230 3770 50  0001 C CNN "LCSC Part"
+F 4 "" H 9230 3770 50  0001 C CNN "LCSC Part"
+F 5 "0" H 9230 3770 50  0001 C CNN "JLCPCB BOM"
 	1    9230 3770
 	1    0    0    -1
@@
 F 2 "Connector_IDC:IDC-Header_2x05_P2.54mm_Vertical" H 1460 1430 50  0001 C CNN
 F 3 "~" H 1460 1430 50  0001 C CNN
-F 4 "0" H 1460 1430 50  0001 C CNN "LCSC Part"
+F 4 "" H 1460 1430 50  0001 C CNN "LCSC Part"
+F 5 "0" H 1460 1430 50  0001 C CNN "JLCPCB BOM"
 	1    1460 1430
 	1    0    0    -1
@@
 F 2 "Connector_IDC:IDC-Header_2x05_P2.54mm_Vertical" H 2730 1430 50  0001 C CNN
 F 3 "~" H 2730 1430 50  0001 C CNN
-F 4 "0" H 2730 1430 50  0001 C CNN "LCSC Part"
+F 4 "" H 2730 1430 50  0001 C CNN "LCSC Part"
+F 5 "0" H 2730 1430 50  0001 C CNN "JLCPCB BOM"
 	1    2730 1430
 	1    0    0    -1
@@
 F 2 "Connector_IDC:IDC-Header_2x05_P2.54mm_Vertical" H 1460 2360 50  0001 C CNN
 F 3 "~" H 1460 2360 50  0001 C CNN
-F 4 "0" H 1460 2360 50  0001 C CNN "LCSC Part"
+F 4 "" H 1460 2360 50  0001 C CNN "LCSC Part"
+F 5 "0" H 1460 2360 50  0001 C CNN "JLCPCB BOM"
 	1    1460 2360
 	1    0    0    -1
@@
 F 2 "Connector_IDC:IDC-Header_2x05_P2.54mm_Vertical" H 2730 2360 50  0001 C CNN
 F 3 "~" H 2730 2360 50  0001 C CNN
-F 4 "0" H 2730 2360 50  0001 C CNN "LCSC Part"
+F 4 "" H 2730 2360 50  0001 C CNN "LCSC Part"
+F 5 "0" H 2730 2360 50  0001 C CNN "JLCPCB BOM"
 	1    2730 2360
 	1    0    0    -1
@@
 F 2 "Connector_IDC:IDC-Header_2x05_P2.54mm_Vertical" H 1430 3250 50  0001 C CNN
 F 3 "~" H 1430 3250 50  0001 C CNN
-F 4 "0" H 1430 3250 50  0001 C CNN "LCSC Part"
+F 4 "" H 1430 3250 50  0001 C CNN "LCSC Part"
+F 5 "0" H 1430 3250 50  0001 C CNN "JLCPCB BOM"
 	1    1430 3250
 	1    0    0    -1
@@
 F 2 "Connector_IDC:IDC-Header_2x05_P2.54mm_Vertical" H 2700 3250 50  0001 C CNN
 F 3 "~" H 2700 3250 50  0001 C CNN
-F 4 "0" H 2700 3250 50  0001 C CNN "LCSC Part"
+F 4 "" H 2700 3250 50  0001 C CNN "LCSC Part"
+F 5 "0" H 2700 3250 50  0001 C CNN "JLCPCB BOM"
 	1    2700 3250
 	1    0    0    -1
@@
 F 2 "Connector_IDC:IDC-Header_2x05_P2.54mm_Vertical" H 1430 4180 50  0001 C CNN
 F 3 "~" H 1430 4180 50  0001 C CNN
-F 4 "0" H 1430 4180 50  0001 C CNN "LCSC Part"
+F 4 "" H 1430 4180 50  0001 C CNN "LCSC Part"
+F 5 "0" H 1430 4180 50  0001 C CNN "JLCPCB BOM"
 	1    1430 4180
 	1    0    0    -1
@@
 F 2 "Connector_IDC:IDC-Header_2x05_P2.54mm_Vertical" H 2700 4180 50  0001 C CNN
 F 3 "~" H 2700 4180 50  0001 C CNN
-F 4 "0" H 2700 4180 50  0001 C CNN "LCSC Part"
+F 4 "" H 2700 4180 50  0001 C CNN "LCSC Part"
+F 5 "0" H 2700 4180 50  0001 C CNN "JLCPCB BOM"
 	1    2700 4180
 	1    0    0    -1
@@
 F 2 "MountingHole:MountingHole_3.2mm_M3_ISO14580_Pad" H 2540 5160 50  0001 C CNN
 F 3 "~" H 2540 5160 50  0001 C CNN
-F 4 "0" H 2540 5160 50  0001 C CNN "LCSC Part"
+F 4 "" H 2540 5160 50  0001 C CNN "LCSC Part"
+F 5 "0" H 2540 5160 50  0001 C CNN "JLCPCB BOM"
 	1    2540 5160
 	0    1    1    0
@@
 F 2 "MountingHole:MountingHole_3.2mm_M3_ISO14580_Pad" H 2540 5340 50  0001 C CNN
 F 3 "~" H 2540 5340 50  0001 C CNN
-F 4 "0" H 2540 5340 50  0001 C CNN "LCSC Part"
+F 4 "" H 2540 5340 50  0001 C CNN "LCSC Part"
+F 5 "0" H 2540 5340 50  0001 C CNN "JLCPCB BOM"
 	1    2540 5340
 	0    1    1    0
@@
 F 2 "MountingHole:MountingHole_3.2mm_M3_ISO14580_Pad" H 2540 5520 50  0001 C CNN
 F 3 "~" H 2540 5520 50  0001 C CNN
-F 4 "0" H 2540 5520 50  0001 C CNN "LCSC Part"
+F 4 "" H 2540 5520 50  0001 C CNN "LCSC Part"
+F 5 "0" H 2540 5520 50  0001 C CNN "JLCPCB BOM"
 	1    2540 5520
 	0    1    1    0
@@
 F 2 "MountingHole:MountingHole_3.2mm_M3_ISO14580_Pad" H 2540 5710 50  0001 C CNN
 F 3 "~" H 2540 5710 50  0001 C CNN
-F 4 "0" H 2540 5710 50  0001 C CNN "LCSC Part"
+F 4 "" H 2540 5710 50  0001 C CNN "LCSC Part"
+F 5 "0" H 2540 5710 50  0001 C CNN "JLCPCB BOM"
 	1    2540 5710
 	0    1    1    0
@@
 F 2 "TerminalBlock_Phoenix:TerminalBlock_Phoenix_MPT-0,5-2-2.54_1x02_P2.54mm_Horizontal" H 4890 1240 50  0001 C CNN
 F 3 "~" H 4890 1240 50  0001 C CNN
-F 4 "0" H 4890 1240 50  0001 C CNN "LCSC Part"
+F 4 "" H 4890 1240 50  0001 C CNN "LCSC Part"
+F 5 "0" H 4890 1240 50  0001 C CNN "JLCPCB BOM"
 	1    4890 1240
 	1    0    0    -1
@@
 F 2 "TerminalBlock_Phoenix:TerminalBlock_Phoenix_MPT-0,5-2-2.54_1x02_P2.54mm_Horizontal" H 4690 2750 50  0001 C CNN
 F 3 "~" H 4690 2750 50  0001 C CNN
-F 4 "0" H 4690 2750 50  0001 C CNN "LCSC Part"
+F 4 "" H 4690 2750 50  0001 C CNN "LCSC Part"
+F 5 "0" H 4690 2750 50  0001 C CNN "JLCPCB BOM"
 	1    4690 2750
 	1    0    0    -1
