File: Alimentation/ModuleMesure/ModuleMesure.kicad_pcb (KiCad board)
At the start: 4 copper layers, 83.5 x 54.8 mm, 71 parts, among them J1 Out Mes 2, J10 I2C SDA, J11 SWD, J12 ARIG Interf, J2 In Mes 1, J3 Out Mes 1, J4 In Mes 2, J5 Out Mes 3, J6 Out Mes 4, J7 In Mes 3, J8 In Mes 4, J9 I2C SCL, Q1 BSS138, Q2 BSS138, SW1 Reset, SW2 Boot0, SW3 Boot1, U1 ACS711xEXLT-15AB, U2 ACS711xEXLT-15AB, U3 ACS711xEXLT-15AB, U4 ACS711xEXLT-15AB, U5 AMS1117-3.3, U6 STM32F103C8Tx, Y1 16Mhz

Commit message: Finalisation pour commande pack Alimentation 14/02/2021
Parts:
- added G***: LOGO, ARIG:Logo_ARIG_12_6x6_6, B.Cu at (155.2, 70.8)
- added G***: LOGO, ARIG:Logo_ARIG_12_6x6_6, F.Cu at (130.0, 61.5)
- moved D2 9.52 mm to (173.2, 65.8)
- moved R14 5.48 mm to (130.8, 82.8), turned to 0 degrees
- moved R11 5.30 mm to (158.5, 82.8), turned to 0 degrees
- moved C3 5.30 mm to (155.0, 85.0), turned to 90 degrees
- moved C4 5.30 mm to (127.2, 85.0), turned to 90 degrees
- moved C1 5.22 mm to (183.8, 70.0), turned to 180 degrees
- moved C2 5.22 mm to (182.8, 85.0), turned to 90 degrees
- moved R21 4.93 mm to (171.0, 65.8), turned to 90 degrees
- moved R10 4.25 mm to (188.0, 82.8), turned to 180 degrees
- moved R9 4.25 mm to (181.5, 64.8), turned to 270 degrees
- moved R2 3.54 mm to (181.0, 71.8), turned to 180 degrees
- moved R4 3.54 mm to (181.0, 82.2), turned to 90 degrees
- moved R6 3.29 mm to (153.2, 82.2), turned to 90 degrees
- moved R8 3.29 mm to (125.5, 82.2), turned to 90 degrees
- moved R1 2.92 mm to (185.0, 71.8)
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Connections:
- U6 pad 10: ANA_CURRENT_1 -> ANA_VOLT_4
- U6 pad 11: ANA_CURRENT_2 -> ANA_CURRENT_4
- U6 pad 12: ANA_CURRENT_3 -> ANA_VOLT_3
- U6 pad 13: ANA_CURRENT_4 -> ANA_CURRENT_3
- U6 pad 14: ANA_VOLT_1 -> ANA_VOLT_2
- U6 pad 15: ANA_VOLT_2 -> ANA_CURRENT_2
- U6 pad 16: ANA_VOLT_3 -> ANA_VOLT_1
- U6 pad 17: ANA_VOLT_4 -> ANA_CURRENT_1
- U6 pad 2: HEART_BEAT -> Net-(U6-Pad2)
- U6 pad 25: FAULT_1 -> FAULT_4
- U6 pad 26: FAULT_2 -> FAULT_3
- U6 pad 27: FAULT_3 -> FAULT_2
- U6 pad 28: FAULT_4 -> FAULT_1
- U6 pad 29: Net-(U6-Pad29) -> HEART_BEAT
Routing:
- net FAULT_4: track 0.00 -> 37.7 mm, vias 0 -> 2
- net ANA_VOLT_4: track 0.00 -> 37.3 mm
- net ANA_CURRENT_1: track 0.00 -> 35.8 mm
- net ANA_CURRENT_4: track 0.00 -> 35.3 mm
- net ANA_VOLT_1: track 0.00 -> 33.5 mm
- net ANA_CURRENT_2: track 0.00 -> 32.1 mm
- net ANA_VOLT_2: track 0.00 -> 30.6 mm
- net FAULT_2: track 0.00 -> 30.0 mm, vias 0 -> 2
- net FAULT_1: track 0.00 -> 23.6 mm
- net GND: track 23.2 -> 45.4 mm, vias 0 -> 14
- net +3V3: track 68.3 -> 86.7 mm, vias 24 -> 33
- net FAULT_3: track 0.00 -> 14.3 mm, vias 0 -> 2
- net +12V: track 0.00 -> 13.0 mm
- net +12L: track 0.00 -> 13.0 mm
- net +12C: track 0.00 -> 13.0 mm
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Other:
- board text added: "Mesure courant Alimentation 2020"

Commit message: Upgrade alim to Kicad 7
Other:
- net class Default removed
