File: Alimentation/ModuleAlim6A/ModuleAlim6A.kicad_sch (KiCad schematic)
At the start: 11 parts, among them J1 Inhibit, J2 Alim. IN / OUT, U1 PTN78020W_EUK-7

Commit message: Upgrade to KicCad 8
Parts:
- U1: footprint ARIG:Texas_EUK_R-PDSS-T7_THT -> Module:Texas_EUK_R-PDSS-T7_THT
