File: Alimentation/MasterAlimCAN/alim.kicad_sch (KiCad schematic)
At the start: 7 parts, among them U10 PTN78020W_EUK-7

Commit message: Init placement for MasterAlimCAN
Parts:
- RV2: renamed from RV1; JLCPCB BOM (none) -> 0
- renumbered C23 to C22, C22 to C25, C25 to C27, F1 to F2

Commit message: New disposition for alim CAN
Parts:
- U10: footprint Module:Texas_EUK_R-PDSS-T7_THT -> ARIG:Texas_EUK_R-PDSS-T7_THT
Changed lines of the file:
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@@
       (effects (font (size 1.27 1.27)))
     )
-    (property "Footprint" "Module:Texas_EUK_R-PDSS-T7_THT" (at 148.59 113.03 0)
+    (property "Footprint" "ARIG:Texas_EUK_R-PDSS-T7_THT" (at 148.59 113.03 0)
       (effects (font (size 1.27 1.27)) hide)
     )
