File: Alimentation/MasterAlimCAN/mesure_lipo.kicad_sch (KiCad schematic)
At the start: 28 parts, among them J14 Lipo Cells, U11 LM358, U6 LM358

Commit message: Finish component placement on MasterAlimCAN
Parts:
- removed J14: Lipo Cells, Connector_PinHeader_2.54mm:PinHeader_1x05_P2.54mm_Vertical, symbol Connector:Conn_01x05_Pin
- added J15: Lipo Cells, Connector_JST:JST_PH_S5B-PH-K_1x05_P2.00mm_Horizontal, symbol Connector_Generic:Conn_01x05
Connections:
- net GND: now also J15.1 (Pin_1)
- net S1: now also J15.2 (Pin_2)
- net S2: now also J15.3 (Pin_3)
- net S3: now also J15.4 (Pin_4)
- net S4: now also J15.5 (Pin_5)
Changed lines of the file:
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@@
+    (stroke (width 0) (type default))
+  )
+  (wire (pts (xy 39.37 74.93) (xy 45.72 74.93))
     (stroke (width 0) (type default))
   )
@@
     (stroke (width 0) (type default))
   )
-  (wire (pts (xy 34.29 69.85) (xy 39.37 69.85))
-    (stroke (width 0) (type default))
-  )
-  (wire (pts (xy 34.29 72.39) (xy 39.37 72.39))
-    (stroke (width 0) (type default))
-  )
   (wire (pts (xy 154.94 36.83) (xy 154.94 30.48))
     (stroke (width 0) (type default))
@@
     (stroke (width 0) (type default))
   )
-  (wire (pts (xy 34.29 74.93) (xy 39.37 74.93))
-    (stroke (width 0) (type default))
-  )
   (wire (pts (xy 171.45 127) (xy 180.34 127))
     (stroke (width 0) (type default))
@@
     (stroke (width 0) (type default))
   )
+  (wire (pts (xy 39.37 77.47) (xy 45.72 77.47))
+    (stroke (width 0) (type default))
+  )
   (wire (pts (xy 158.75 92.71) (xy 158.75 83.82))
     (stroke (width 0) (type default))
@@
     (stroke (width 0) (type default))
   )
-  (wire (pts (xy 34.29 77.47) (xy 39.37 77.47))
-    (stroke (width 0) (type default))
-  )
   (wire (pts (xy 176.53 81.28) (xy 180.34 81.28))
     (stroke (width 0) (type default))
@@
     (stroke (width 0) (type default))
   )
+  (wire (pts (xy 36.83 67.31) (xy 45.72 67.31))
+    (stroke (width 0) (type default))
+  )
   (wire (pts (xy 187.96 81.28) (xy 190.5 81.28))
     (stroke (width 0) (type default))
@@
     (stroke (width 0) (type default))
   )
-  (wire (pts (xy 34.29 67.31) (xy 36.83 67.31))
+  (wire (pts (xy 39.37 69.85) (xy 45.72 69.85))
     (stroke (width 0) (type default))
   )
@@
   )
   (wire (pts (xy 156.21 83.82) (xy 158.75 83.82))
+    (stroke (width 0) (type default))
+  )
+  (wire (pts (xy 39.37 72.39) (xy 45.72 72.39))
     (stroke (width 0) (type default))
   )
@@
     )
   )
+  (symbol (lib_id "Connector_Generic:Conn_01x05") (at 50.8 72.39 0) (unit 1)
+    (in_bom yes) (on_board yes) (dnp no) (fields_autoplaced)
+    (property "Reference" "J15" (at 53.34 71.12 0)
+      (effects (font (size 1.27 1.27)) (justify left))
+    )
+    (property "Value" "Lipo Cells" (at 53.34 73.66 0)
+      (effects (font (size 1.27 1.27)) (justify left))
+    )
+    (property "Footprint" "Connector_JST:JST_PH_S5B-PH-K_1x05_P2.00mm_Horizontal" (at 50.8 72.39 0)
+      (effects (font (size 1.27 1.27)) hide)
+    )
+    (property "Datasheet" "~" (at 50.8 72.39 0)
+      (effects (font (size 1.27 1.27)) hide)
+    )
+    (property "JLCPCB BOM" "0" (at 50.8 72.39 0)
+      (effects (font (size 1.27 1.27)) hide)
+    )
+    (pin "1")
+    (pin "4")
+    (pin "5")
+    (pin "3")
+    (pin "2")
+    (instances
+      (project "MasterAlimCAN"
+        (path "/c83bc042-587c-48f9-abdb-41233c8ec938/1021524a-f267-4cff-8043-52ba598edf0c"
+          (reference "J15") (unit 1)
+        )
+      )
+    )
+  )
   (symbol (lib_id "Amplifier_Operational:LM358") (at 97.79 113.03 0) (unit 2)
     (in_bom yes) (on_board yes) (dnp no) (fields_autoplaced)
@@
         )
       )
-    )
-  )
-  (symbol (lib_id "Connector:Conn_01x05_Pin") (at 29.21 72.39 0) (unit 1)
-    (in_bom yes) (on_board yes) (dnp no)
-    (property "Reference" "J14" (at 31.75 60.96 0)
-      (effects (font (size 1.27 1.27)))
-    )
-    (property "Value" "Lipo Cells" (at 31.75 63.5 0)
-      (effects (font (size 1.27 1.27)))
-    )
-    (property "Footprint" "Connector_PinHeader_2.54mm:PinHeader_1x05_P2.54mm_Vertical" (at 29.21 72.39 0)
-      (effects (font (size 1.27 1.27)) hide)
-    )
-    (property "Datasheet" "~" (at 29.21 72.39 0)
-      (effects (font (size 1.27 1.27)) hide)
-    )
-    (property "JLCPCB BOM" "0" (at 29.21 72.39 0)
-      (effects (font (size 1.27 1.27)) hide)
-    )
-    (pin "1")
-    (pin "5")
-    (pin "3")
-    (pin "4")
-    (pin "2")
-    (instances
-      (project "MasterAlimCAN"
-        (path "/c83bc042-587c-48f9-abdb-41233c8ec938/1021524a-f267-4cff-8043-52ba598edf0c"
-          (reference "J14") (unit 1)
-        )
-      )
