File: ControlleursAsserv/ControlleursAsserv.kicad_pcb (KiCad board)
At the start: 4 copper layers, 85 x 56 mm, 101 parts, among them J1 I2C1_5, J10 Codeur, J11 Motor FeedBack, J12 Motor CMD, J13 Codeur, J14 Motor FeedBack, J15 Motor CMD, J16 Codeur, J17 Motor FeedBack, J18 Motor CMD, J2 I2C2_5, J3 CAN1, J4 CAN2, J5 In App Prog, J6 DEBUG, J7 Codeur, J8 Motor CMD, J9 Motor FeedBack, Q1 BSS138, Q10 BSS138, Q11 BSS138, Q12 BSS138, Q13 BSS138, Q14 BSS138, Q2 BSS138, Q3 BSS138, Q4 BSS138, Q5 BSS138, Q6 BSS138, Q7 BSS138, Q8 BSS138, Q9 BSS138, SW1 RESET, SW2 BOOT0, U1 STM32G474RETx, U2 AMS1117-3.3, U3 MCP2558FD-xSN, Y1 16MHz

Commit message: Generate all production files
Parts:
- added G***: LOGO, ARIG:Logo_ARIG_12_6x6_6, B.Cu at (100.2, 90.5)
Other:
- board text added: "Boot 0"
- board text added: "Codeur 1"
- board text added: "Codeur 2"
- board text added: "Codeur 3"
- board text added: "Codeur 4"
- board text added: "Controlleur Asserv 2024"
- board text added: "FB 1"
- board text added: "FB 2"
- board text added: "FB 3"
- board text added: "FB 4"
- board text added: "H.B."
- board text added: "Moteur 1"
- board text added: "Moteur 2"
- board text added: "Moteur 3"
- board text added: "Moteur 4"
- board text added: "PWR"
- board text added: "Reset"
