File: InterfaceMotorPami/InterfaceMotorPami.kicad_pcb (KiCad board)
At the start: 2 copper layers, 31.3 x 25.5 mm, 5 parts, among them J1 MOT, J2 PONT H, J3 Codeur

Commit message: Generate all production files
Changed lines of the file:
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@@
 			(layers "*.Cu" "*.Mask")
 			(remove_unused_layers no)
-			(roundrect_rratio 0.147059)
+			(roundrect_rratio 0.1470588235)
 			(net 5 "/MOT-")
 			(pinfunction "Pin_1")
@@
 			(layers "*.Cu" "*.Mask")
 			(remove_unused_layers no)
-			(roundrect_rratio 0.208333)
+			(roundrect_rratio 0.2083333333)
 			(net 6 "+5V")
 			(pinfunction "Pin_1")
