File: InterfaceRaspiCAN/level_shifter.kicad_sch (KiCad schematic)
At the start: 3 parts, among them Q1 BSS138

Commit message: Add PCB for RaspiCAN
Parts:
- R2, R3: footprint (none) -> Resistor_SMD:R_0805_2012Metric_Pad1.20x1.40mm_HandSolder
Changed lines of the file:
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@@
       (effects (font (size 1.27 1.27)) (justify left))
     )
-    (property "Footprint" "" (at 125.222 88.9 90)
+    (property "Footprint" "Resistor_SMD:R_0805_2012Metric_Pad1.20x1.40mm_HandSolder" (at 125.222 88.9 90)
       (effects (font (size 1.27 1.27)) hide)
     )
@@
       (effects (font (size 1.27 1.27)) (justify left))
     )
-    (property "Footprint" "" (at 143.002 88.9 90)
+    (property "Footprint" "Resistor_SMD:R_0805_2012Metric_Pad1.20x1.40mm_HandSolder" (at 143.002 88.9 90)
       (effects (font (size 1.27 1.27)) hide)
     )

Commit message: Generate all production files
Parts:
- Q1: LCSC Part (none) -> C426569
- R2, R3: LCSC Part (none) -> C17414
Changed lines of the file:
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@@
+			)
+		)
+		(property "LCSC Part" "C17414"
+			(at 127 88.9 0)
+			(effects
+				(font
+					(size 1.27 1.27)
+				)
+				(hide yes)
 			)
 		)
@@
 		)
 		(property "Description" "50V Vds, 0.22A Id, N-Channel MOSFET, SOT-23"
+			(at 137.16 93.98 0)
+			(effects
+				(font
+					(size 1.27 1.27)
+				)
+				(hide yes)
+			)
+		)
+		(property "LCSC Part" "C426569"
 			(at 137.16 93.98 0)
 			(effects
@@
 			(at 144.78 88.9 0)
 			(effects
+				(font
+					(size 1.27 1.27)
+				)
+				(hide yes)
+			)
+		)
+		(property "LCSC Part" "C17414"
+			(at 144.78 88.9 0)
+			(effects
